Commit message: Update robotiq.ros2_control.xacro

File: ur_description/urdf/ur5e/robotiq.ros2_control.xacro (robot description, xacro)
@@ -71,119 +71,4 @@
       <xacro:configure_joint joint_name="${tf_prefix}robotiq_85_right_finger_tip_joint"
         mimicing_joint="${tf_prefix}robotiq_85_left_knuckle_joint" multiplier="-1" />
-      <!-- <joint name="${tf_prefix}robotiq_85_left_knuckle_joint">
-        <xacro:unless value="${ros2_control_hardware_type == 'mujoco'}">
-          <param name="position_kp">3000</param>
-          <param name="position_ki">1</param>
-          <param name="position_kd">100</param>
-          <param name="position_i_max">10000</param>
-          <command_interface name="position_pid" />
-        </xacro:unless>
-        <xacro:if value="${ros2_control_hardware_type == 'mujoco'}">
-          <command_interface name="position" />
-        </xacro:if>
-        <state_interface name="position">
-          <param name="initial_value">${initial_positions['robotiq_85_left_knuckle_joint']}</param>
-        </state_interface>
-        <state_interface name="velocity">
-          <param name="initial_value">0.0</param>
-        </state_interface>
-      </joint>
-      <joint name="${tf_prefix}robotiq_85_right_knuckle_joint">
-        <param name="mimic">${tf_prefix}robotiq_85_left_knuckle_joint</param>
-        <xacro:unless value="${ros2_control_hardware_type == 'mujoco'}">
-          <param name="position_kp">3000</param>
-          <param name="position_ki">1</param>
-          <param name="position_kd">100</param>
-          <param name="position_i_max">10000</param>
-          <command_interface name="position_pid" />
-        </xacro:unless>
-        <xacro:if value="${ros2_control_hardware_type == 'mujoco'}">
-          <command_interface name="position" />
-        </xacro:if>
-        <state_interface name="position">
-          <param name="initial_value">0.0</param>
-        </state_interface>
-        <state_interface name="velocity">
-          <param name="initial_value">0.0</param>
-        </state_interface>
-      </joint>
-      <joint name="${tf_prefix}robotiq_85_left_inner_knuckle_joint">
-        <param name="mimic">${tf_prefix}robotiq_85_left_knuckle_joint</param>
-        <xacro:unless value="${ros2_control_hardware_type == 'mujoco'}">
-          <param name="position_kp">3000</param>
-          <param name="position_ki">1</param>
-          <param name="position_kd">100</param>
-          <param name="position_i_max">10000</param>
-          <command_interface name="position_pid" />
-        </xacro:unless>
-        <xacro:if value="${ros2_control_hardware_type == 'mujoco'}">
-          <command_interface name="position" />
-        </xacro:if>
-        <state_interface name="position">
-          <param name="initial_value">0.0</param>
-        </state_interface>
-        <state_interface name="velocity">
-          <param name="initial_value">0.0</param>
-        </state_interface>
-      </joint>
-      <joint name="${tf_prefix}robotiq_85_right_inner_knuckle_joint">
-        <param name="mimic">${tf_prefix}robotiq_85_left_knuckle_joint</param>
-        <xacro:unless value="${ros2_control_hardware_type == 'mujoco'}">
-          <param name="position_kp">3000</param>
-          <param name="position_ki">1</param>
-          <param name="position_kd">100</param>
-          <param name="position_i_max">10000</param>
-          <command_interface name="position_pid" />
-        </xacro:unless>
-        <xacro:if value="${ros2_control_hardware_type == 'mujoco'}">
-          <command_interface name="position" />
-        </xacro:if>
-        <state_interface name="position">
-          <param name="initial_value">0.0</param>
-        </state_interface>
-        <state_interface name="velocity">
-          <param name="initial_value">0.0</param>
-        </state_interface>
-      </joint>
-      <joint name="${tf_prefix}robotiq_85_right_finger_tip_joint">
-        <param name="mimic">${tf_prefix}robotiq_85_left_knuckle_joint</param>
-        <param name="multiplier">-1</param>
-        <xacro:unless value="${ros2_control_hardware_type == 'mujoco'}">
-          <param name="position_kp">3000</param>
-          <param name="position_ki">1</param>
-          <param name="position_kd">100</param>
-          <param name="position_i_max">10000</param>
-          <command_interface name="position_pid" />
-        </xacro:unless>
-        <xacro:if value="${ros2_control_hardware_type == 'mujoco'}">
-          <command_interface name="position" />
-        </xacro:if>
-        <state_interface name="position">
-          <param name="initial_value">0.0</param>
-        </state_interface>
-        <state_interface name="velocity">
-          <param name="initial_value">0.0</param>
-        </state_interface>
-      </joint>
-      <joint name="${tf_prefix}robotiq_85_left_finger_tip_joint">
-        <param name="mimic">${tf_prefix}robotiq_85_left_knuckle_joint</param>
-        <param name="multiplier">-1</param>
-        <xacro:unless value="${ros2_control_hardware_type == 'mujoco'}">
-          <param name="position_kp">3000</param>
-          <param name="position_ki">1</param>
-          <param name="position_kd">100</param>
-          <param name="position_i_max">10000</param>
-          <command_interface name="position_pid" />
-        </xacro:unless>
-        <xacro:if value="${ros2_control_hardware_type == 'mujoco'}">
-          <command_interface name="position" />
-        </xacro:if>
-        <state_interface name="position">
-          <param name="initial_value">0.0</param>
-        </state_interface>
-        <state_interface name="velocity">
-          <param name="initial_value">0.0</param>
-        </state_interface>
-      </joint> -->
     </ros2_control>
   </xacro:macro>
